Commit message: The updated xacro and gazebo files

File: urdf/robot.xacro (robot description, xacro)
@@ -76,5 +76,30 @@
     </visual>
   </link>
-  <link name="neck_link">
+   <link name="link_right_wheel">
+    <xacro:default_inertial mass="0.2"/>
+    <collision name="link_right_wheel_collision">
+      <origin rpy="0 1.5707 1.5707" xyz="0 0 0"/>
+      <xacro:wheel_geometry />
+    </collision>
+    <visual name="link_right_wheel_visual">
+      <origin rpy="0 1.5707 1.5707" xyz="0 0 0"/>
+      <xacro:wheel_geometry />
+      <material name="red"/>
+    </visual>
+  </link>
+   <link name="link_left_wheel">
+    <xacro:default_inertial mass="0.2"/>
+    <collision name="link_left_wheel_collision">
+      <origin rpy="0 1.5707 1.5707" xyz="0 0 0"/>
+      <xacro:wheel_geometry />
+    </collision>
+    <visual name="link_left_wheel_visual">
+      <origin rpy="0 1.5707 1.5707" xyz="0 0 0"/>
+      <xacro:wheel_geometry />
+      <material name="red"/>
+    </visual>
+  </link>
+  <!-- neck link -->
+  <link name="link_neck">
   	<inertial>
 	<mass value="0.025"/>
@@ -96,5 +121,6 @@
   	</visual>
   </link>
-  <link name="head_link">
+  <!-- link of head -->
+  <link name="link_head">
   	<inertial>
 	<mass value="0.025"/>
@@ -116,28 +142,4 @@
   	</visual>
   </link>
-   <link name="link_right_wheel">
-    <xacro:default_inertial mass="0.2"/>
-    <collision name="link_right_wheel_collision">
-      <origin rpy="0 1.5707 1.5707" xyz="0 0 0"/>
-      <xacro:wheel_geometry />
-    </collision>
-    <visual name="link_right_wheel_visual">
-      <origin rpy="0 1.5707 1.5707" xyz="0 0 0"/>
-      <xacro:wheel_geometry />
-      <material name="red"/>
-    </visual>
-  </link>
-   <link name="link_left_wheel">
-    <xacro:default_inertial mass="0.2"/>
-    <collision name="link_left_wheel_collision">
-      <origin rpy="0 1.5707 1.5707" xyz="0 0 0"/>
-      <xacro:wheel_geometry />
-    </collision>
-    <visual name="link_left_wheel_visual">
-      <origin rpy="0 1.5707 1.5707" xyz="0 0 0"/>
-      <xacro:wheel_geometry />
-      <material name="red"/>
-    </visual>
-  </link>
   <link name="camera_link">
     <collision>
@@ -162,12 +164,4 @@
     </inertial>
   </link>
-<!--************************************JOINTS****************************************-->
-  <joint name="head_joint" type="revolute">
-  	<axis xyz="0 0 1"/>
-  	<limit effort="1000.0" lower="-3.14" upper="3.14" velocity="0.2"/>
-  	<origin rpy="0 0 0" xyz="0 0 0"/>
-  	<parent link="neck_link"/>
-  	<child link="head_link"/>
-  </joint>
   <joint name="joint_right_wheel" type="continuous">
     <origin rpy="0 0 0" xyz="-0.05 0.15 0"/>
@@ -186,19 +180,26 @@
     <joint_properties damping="1.0" friction="1.0"/>
   </joint>
-  <joint name="neck_joint" type="fixed">
+  <joint name="joint_neck" type="fixed">
   	<origin rpy="0 0 0" xyz="0.26 0 0"/> <!--0.06-->
   	<parent link="link_chassis"/>
-  	<child link="neck_link"/>
+  	<child link="link_neck"/>
+  </joint>
+    <joint name="joint_head" type="revolute">
+  	<axis xyz="0 0 1"/>
+  	<limit effort="1000.0" lower="-3.14" upper="3.14" velocity="0.2"/>
+  	<origin rpy="0 0 0" xyz="0 0 0"/>
+  	<parent link="link_neck"/>
+  	<child link="link_head"/>
   </joint>
   <joint name="camera_joint" type="fixed">
 	    <axis xyz="1 0 0" />
 	    <origin xyz="0 0 0" rpy="0 0 0"/>
-	    <parent link="head_link"/>
+	    <parent link="link_head"/>
 	    <child link="camera_link"/>
   </joint>
-<!--************************************TRANSMISSION****************************************-->
+<!--Transmission-->
 <transmission name="head_joint_trans">
 	<type>transmission_interface/SimpleTransmission</type>
-	<joint name="head_joint">
+	<joint name="joint_head">
 		<hardwareInterface>hardware_interface/EffortJointInterface</hardwareInterface>
 	</joint>
